Commit message: Added xeno_can_test.cpp to debugg CAN bus connectivity

File: xeno_interface/models/xeno.xacro (robot description, xacro)
@@ -29,11 +29,11 @@
     <xacro:property name="right_arm_length" value="0.45" />
     <xacro:property name="arm_offset_vertical" value="0.18" />
-	<xacro:property name="arm_z_offset" value="0.096" />
-	<!-- Main base prism -->
-	<xacro:property name="robot_base_length" value="0.838" />
-	<xacro:property name="robot_base_width" value="0.49" />
-	<xacro:property name="robot_base_height" value="0.404" />
-	<xacro:property name="robot_base_z_offset"
-					value="${front_wheel_diameter / 2.0}" />
+    <xacro:property name="arm_z_offset" value="0.096" />
+    <!-- Main base prism -->
+    <xacro:property name="robot_base_length" value="0.838" />
+    <xacro:property name="robot_base_width" value="0.49" />
+    <xacro:property name="robot_base_height" value="0.404" />
+    <xacro:property name="robot_base_z_offset"
+		    value="${front_wheel_diameter / 2.0}" />
 	<!-- footrest -->
     <xacro:property name="footrest_length" value="0.2" />
@@ -44,22 +44,22 @@
     <xacro:property name="camera_pole_height" value="${1.12 + 0.06}" />
     <xacro:property name="camera_pole_diameter" value="0.039" />
-	<xacro:property name="camera_mount_length" value="0.28" />
-	<xacro:property name="camera_pole_x_offset" value="0.0" />
-	<xacro:property name="camera_pole_y_offset" value="0.019" />
-	<!-- Seat cusion -->
-	<xacro:property name="seat_cusion_height" value="0.05" />
-	<xacro:property name="seat_cusion_width" value="0.44" />
-	<xacro:property name="seat_cusion_length" value="0.44" />
-	<xacro:property name="seat_x_offset" value="0.05" />
-	<xacro:macro name="color_black">
+    <xacro:property name="camera_mount_length" value="0.28" />
+    <xacro:property name="camera_pole_x_offset" value="0.0" />
+    <xacro:property name="camera_pole_y_offset" value="0.019" />
+    <!-- Seat cusion -->
+    <xacro:property name="seat_cusion_height" value="0.05" />
+    <xacro:property name="seat_cusion_width" value="0.44" />
+    <xacro:property name="seat_cusion_length" value="0.44" />
+    <xacro:property name="seat_x_offset" value="0.05" />
+    <xacro:macro name="color_black">
       <material name="black">
         <color rgba="0.3 0.3 0.4 1.0" />
       </material>
-	</xacro:macro>
-	<xacro:macro name="color_orange">
+    </xacro:macro>
+    <xacro:macro name="color_orange">
       <material name="orange">
         <color rgba="1.0 0.5 0 1.0" />
       </material>
-	</xacro:macro>
+    </xacro:macro>
     <xacro:macro name="color_gray">
       <material name="gray">
@@ -67,5 +67,5 @@
       </material>
     </xacro:macro>
-	<xacro:macro name="color_darkgray1">
+    <xacro:macro name="color_darkgray1">
       <material name="dark_gray">
         <color rgba="0.4 0.4 0.5 1.0" />
@@ -73,11 +73,11 @@
     </xacro:macro>
 	<!-- useful macros -->
-    <xacro:macro name="prism" params="name x y z *color">
-      <link name="${name}">
-        <visual>
-          <geometry>
-            <box size="${x} ${y} ${z}" />
-          </geometry>
-          <xacro:insert_block name="color" />
+	<xacro:macro name="prism" params="name x y z *color">
+	  <link name="${name}">
+            <visual>
+              <geometry>
+		<box size="${x} ${y} ${z}" />
+              </geometry>
+              <xacro:insert_block name="color" />
         </visual>
         <collision>
@@ -86,228 +86,228 @@
           </geometry>
         </collision>
-      </link>
-    </xacro:macro>
-    <xacro:macro name="cyl" params="name radius length *color">
-        <link name="${name}">
+	  </link>
+	</xacro:macro>
+	<xacro:macro name="cyl" params="name radius length *color">
+          <link name="${name}">
             <visual>
-                <geometry>
-                    <cylinder radius="${radius}" length="${length}" />
-                </geometry>
-                <xacro:insert_block name="color" />
+              <geometry>
+                <cylinder radius="${radius}" length="${length}" />
+              </geometry>
+              <xacro:insert_block name="color" />
             </visual>
             <collision>
-                <geometry>
-                    <cylinder radius="${radius}" length="${length}" />
-                </geometry>
+              <geometry>
+                <cylinder radius="${radius}" length="${length}" />
+              </geometry>
             </collision>
-        </link>
-    </xacro:macro>
-    <!-- end useful macros -->
+          </link>
+	</xacro:macro>
+	<!-- end useful macros -->
 	<!-- Building up the robot -->
 	<link name="base_footprint" />
 	<joint name="base_footprint_to_base_link" type="fixed">
-      <parent link="base_footprint" />
-      <child link="base_link" />
+	  <parent link="base_footprint" />
+	  <child link="base_link" />
       <origin
           xyz="0 0 ${rear_wheel_diameter / 2.0}"
           rpy="0 0 0" />
     </joint>
-	<link name="base_link" />
-	<joint name="base_link_to_base" type="fixed">
-      <parent link="base_link" />
-      <child link="base" />
-      <origin
-          xyz="${rear_wheel_diameter / 2.0} 0.0
-			   ${robot_base_z_offset + (robot_base_height / 2.0)
-			   - (rear_wheel_diameter / 2.0) }"
-          rpy="0 0 0" />
-    </joint>
-	<xacro:prism
-        name="base"
-        x="${robot_base_length}"
-        y="${robot_base_width}"
-        z="${robot_base_height}">
-      <xacro:color_orange />
-    </xacro:prism>
-	<xacro:prism
-        name="seat_cusion"
-        x="${seat_cusion_length}"
-        y="${seat_cusion_width}"
-        z="${seat_cusion_height}">
-      <xacro:color_black />
-    </xacro:prism>
-	<joint name="base_to_seat_cusion" type="fixed">
-		<parent link="base" />
-		<child link="seat_cusion" />
-		<origin
-			xyz="${seat_x_offset} 0 ${robot_base_height / 2 + seat_cusion_height
-				 / 2}"
-			rpy="0 0 0" />
-		<axis xyz="1 0 0" />
-	  </joint>
-	<xacro:macro name="rear_wheel" params="name side_mult">
-	  <xacro:cyl
-          name="rear_${name}_wheel"
-          radius="${rear_wheel_diameter / 2}"
-          length="${rear_wheel_thickness}">
-        <xacro:color_gray />
-      </xacro:cyl>
-      <joint name="wheelchair_base_to_rear_${name}_wheel" type="fixed">
-        <parent link="base" />
-        <child link="rear_${name}_wheel" />
-        <origin
-            xyz="${-robot_base_length/2 + rear_wheel_axis_offset}
-				 ${side_mult * (robot_base_width + rear_wheel_thickness) / 2.0}
-				 ${-robot_base_height/2.0 + (rear_wheel_diameter -
-				 front_wheel_diameter) /2.0}"
-            rpy="${-halfpi * side_mult} 0 0" />
-        <axis xyz="1 0 0" />
-      </joint>
-	</xacro:macro>
-	<xacro:macro name="front_wheel" params="name side_mult">
-	  <!-- Wheel -->
-	  <xacro:cyl
-		  name="front_${name}_wheel"
-		  radius="${front_wheel_diameter / 2}"
-		  length="${front_wheel_thickness}">
-		<xacro:color_gray />
-	  </xacro:cyl>
-	  <joint name="base_to_front_${name}_wheel" type="fixed">
-		<parent link="base" />
-		<child link="front_${name}_wheel" />
-		<origin
-			xyz="${robot_base_length/2} ${side_mult * (robot_base_width +
-				 rear_wheel_thickness) / 2.0}
-				 ${-robot_base_height/2.0}"
-			rpy="${-halfpi * side_mult} 0 0" />
-		<axis xyz="1 0 0" />
-	  </joint>
-	</xacro:macro>
-	<xacro:rear_wheel
-		name="left"
-		side_mult="1" />
-	<xacro:rear_wheel
-		name="right"
-		side_mult="-1" />
-	<xacro:front_wheel
-		name="left"
-		side_mult="1" />
-	<xacro:front_wheel
-		name="right"
-		side_mult="-1" />
-	    <xacro:prism
-        name="upright"
-        x="${backrest_thickness}"
-        y="${backrest_width}"
-        z="${backrest_height}">
-        <xacro:color_black />
-    </xacro:prism>
-    <joint name="upright_joint" type="fixed">
-        <parent link="base" />
-        <child link="upright" />
-        <origin
-            xyz="${-(robot_base_length / 2) + backrest_thickness / 2
-				 + 	rear_wheel_axis_offset + backrest_x_offset}
-				 0
-				 ${(robot_base_height / 2) + (backrest_height / 2)}"
-            rpy="0 0 0" />
-    </joint>
-	<!-- Left arm of the wheelchair, does not have the joystick -->
-    <xacro:prism
-        name="left_armrest"
-        x="${left_arm_length}"
-        y="${arm_width}"
-        z="${arm_height}">
-        <xacro:color_darkgray1 />
-    </xacro:prism>
-    <joint name="left_arm_joint" type="fixed">
-        <parent link="upright" />
-        <child link="left_armrest" />
-        <origin
-            xyz="${(left_arm_length + backrest_thickness) / 2 + arm_z_offset} ${(arm_width + backrest_width) / 2} ${-(backrest_height) / 2 + arm_offset_vertical}"
-            rpy="0 0 0" />
-    </joint>
-	<!-- Right arm of the wheelchair, includes the joystick-->
-	<xacro:prism
-        name="right_armrest"
-        x="${right_arm_length}"
-        y="${arm_width}"
-        z="${arm_height}">
-      <xacro:color_darkgray1 />
-    </xacro:prism>
-    <joint name="right_arm_joint" type="fixed">
-      <parent link="upright" />
-      <child link="right_armrest" />
-      <origin
-          xyz="${(right_arm_length + backrest_thickness) / 2 + arm_z_offset}
-			   ${-(arm_width + backrest_width) / 2}
-			   ${-(backrest_height) / 2 + arm_offset_vertical}"
-          rpy="0 0 0" />
-    </joint>
+    <link name="base_link" />
+    <!-- <joint name="base_link_to_base" type="fixed"> -->
+    <!--   <parent link="base_link" /> -->
+    <!--   <child link="base" /> -->
+    <!--   <origin -->
+    <!--       xyz="${rear_wheel_diameter / 2.0} 0.0 -->
+    <!-- 			   ${robot_base_z_offset + (robot_base_height / 2.0) -->
+    <!-- 			   - (rear_wheel_diameter / 2.0) }" -->
+    <!--       rpy="0 0 0" /> -->
+    <!-- </joint> -->
+    <!-- <xacro:prism -->
+    <!--     name="base" -->
+    <!--     x="${robot_base_length}" -->
+    <!--     y="${robot_base_width}" -->
+    <!--     z="${robot_base_height}"> -->
+    <!--   <xacro:color_orange /> -->
+    <!-- </xacro:prism> -->
+    <!-- 	<xacro:prism -->
+    <!--     name="seat_cusion" -->
+    <!--     x="${seat_cusion_length}" -->
+    <!--     y="${seat_cusion_width}" -->
+    <!--     z="${seat_cusion_height}"> -->
+    <!--   <xacro:color_black /> -->
+    <!-- </xacro:prism> -->
+    <!-- 	<joint name="base_to_seat_cusion" type="fixed"> -->
+    <!-- 		<parent link="base" /> -->
+    <!-- 		<child link="seat_cusion" /> -->
+    <!-- 		<origin -->
+    <!-- 			xyz="${seat_x_offset} 0 ${robot_base_height / 2 + seat_cusion_height -->
+    <!-- 				 / 2}" -->
+    <!-- 			rpy="0 0 0" /> -->
+    <!-- 		<axis xyz="1 0 0" /> -->
+    <!-- 	  </joint>	  	   -->
+      <!-- 	<xacro:macro name="rear_wheel" params="name side_mult"> -->
+      <!-- 	  <xacro:cyl -->
+      <!--     name="rear_${name}_wheel" -->
+      <!--     radius="${rear_wheel_diameter / 2}" -->
+      <!--     length="${rear_wheel_thickness}"> -->
+      <!--   <xacro:color_gray /> -->
+      <!-- </xacro:cyl> -->
+    <!--   <joint name="wheelchair_base_to_rear_${name}_wheel" type="fixed"> -->
+    <!--     <parent link="base" /> -->
+    <!--     <child link="rear_${name}_wheel" /> -->
+    <!--     <origin -->
+    <!--         xyz="${-robot_base_length/2 + rear_wheel_axis_offset} -->
+    <!-- 				 ${side_mult * (robot_base_width + rear_wheel_thickness) / 2.0} -->
+    <!-- 				 ${-robot_base_height/2.0 + (rear_wheel_diameter - -->
+    <!-- 				 front_wheel_diameter) /2.0}"  -->
+    <!--         rpy="${-halfpi * side_mult} 0 0" /> -->
+    <!--     <axis xyz="1 0 0" /> -->
+    <!--   </joint>	   -->
+    <!-- 	</xacro:macro> -->
+    <!-- 	<xacro:macro name="front_wheel" params="name side_mult"> -->
+    <!-- Wheel -->
+    <!-- 	  <xacro:cyl -->
+    <!-- 		  name="front_${name}_wheel" -->
+    <!-- 		  radius="${front_wheel_diameter / 2}" -->
+    <!-- 		  length="${front_wheel_thickness}"> -->
+    <!-- 		<xacro:color_gray />				 -->
+    <!-- 	  </xacro:cyl> -->
+    <!-- 	  <joint name="base_to_front_${name}_wheel" type="fixed"> -->
+    <!-- 		<parent link="base" /> -->
+    <!-- 		<child link="front_${name}_wheel" /> -->
+    <!-- 		<origin -->
+    <!-- 			xyz="${robot_base_length/2} ${side_mult * (robot_base_width + -->
+    <!-- 				 rear_wheel_thickness) / 2.0} -->
+    <!-- 				 ${-robot_base_height/2.0}" -->
+    <!-- 			rpy="${-halfpi * side_mult} 0 0" /> -->
+    <!-- 		<axis xyz="1 0 0" /> -->
+    <!-- 	  </joint>	  	   -->
+    <!-- 	</xacro:macro> -->
+    <!-- 	<xacro:rear_wheel -->
+    <!-- 		name="left" -->
+    <!-- 		side_mult="1" /> -->
+    <!-- 	<xacro:rear_wheel -->
+    <!-- 		name="right" -->
+    <!-- 		side_mult="-1" /> -->
+    <!-- 	<xacro:front_wheel -->
+    <!-- 		name="left" -->
+    <!-- 		side_mult="1" /> -->
+    <!-- 	<xacro:front_wheel -->
+    <!-- 		name="right" -->
+    <!-- 		side_mult="-1" /> -->
+    <!-- 	    <xacro:prism -->
+    <!--     name="upright" -->
+    <!--     x="${backrest_thickness}" -->
+    <!--     y="${backrest_width}" -->
+    <!--     z="${backrest_height}"> -->
+    <!--     <xacro:color_black /> -->
+    <!-- </xacro:prism> -->
+    <!-- <joint name="upright_joint" type="fixed"> -->
+    <!--     <parent link="base" /> -->
+    <!--     <child link="upright" /> -->
+    <!--     <origin -->
+    <!--         xyz="${-(robot_base_length / 2) + backrest_thickness / 2 -->
+    <!-- 				 + 	rear_wheel_axis_offset + backrest_x_offset}  -->
+    <!-- 				 0 -->
+    <!-- 				 ${(robot_base_height / 2) + (backrest_height / 2)}" -->
+    <!--         rpy="0 0 0" /> -->
+    <!-- </joint> -->
+    <!-- Left arm of the wheelchair, does not have the joystick -->
+    <!-- <xacro:prism -->
+    <!--     name="left_armrest" -->
+    <!--     x="${left_arm_length}" -->
+    <!--     y="${arm_width}" -->
+    <!--     z="${arm_height}"> -->
+    <!--     <xacro:color_darkgray1 /> -->
+    <!-- </xacro:prism> -->
+    <!-- <joint name="left_arm_joint" type="fixed"> -->
+    <!--     <parent link="upright" /> -->
+    <!--     <child link="left_armrest" /> -->
+    <!--     <origin -->
+    <!--         xyz="${(left_arm_length + backrest_thickness) / 2 + arm_z_offset} ${(arm_width + backrest_width) / 2} ${-(backrest_height) / 2 + arm_offset_vertical}" -->
+    <!--         rpy="0 0 0" /> -->
+    <!-- </joint> -->
+    <!-- Right arm of the wheelchair, includes the joystick-->
+    <!-- 	<xacro:prism -->
+    <!--     name="right_armrest" -->
+    <!--     x="${right_arm_length}" -->
+    <!--     y="${arm_width}" -->
+    <!--     z="${arm_height}"> -->
+    <!--   <xacro:color_darkgray1 /> -->
+    <!-- </xacro:prism> -->
+    <!-- <joint name="right_arm_joint" type="fixed"> -->
+    <!--   <parent link="upright" /> -->
+    <!--   <child link="right_armrest" /> -->
+    <!--   <origin -->
+    <!--       xyz="${(right_arm_length + backrest_thickness) / 2 + arm_z_offset} -->
+    <!-- 			   ${-(arm_width + backrest_width) / 2} -->
+    <!-- 			   ${-(backrest_height) / 2 + arm_offset_vertical}" -->
+    <!--       rpy="0 0 0" /> -->
+    <!-- </joint> -->
     <!-- footrest -->
-    <xacro:prism
-        name="footrest"
-        x="${footrest_length}"
-        y="${footrest_width}"
-        z="${footrest_height}">
-        <xacro:color_black />
-    </xacro:prism>
-    <joint name="footrest_joint" type="fixed">
-        <parent link="base" />
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